Commit message: 🗃️[Mod] 차량 URDF 수정

File: src/my_slam/urdf/robot.urdf (robot description, URDF)
Before this commit: robot my_robot, 7 links, 6 joints
Links:
- added link rear_wheel_axis; visual box size=0.02 0.12 0.02
- added link steering_link; visual box size=0.02 0.12 0.02
- link front_left_wheel: geometry visual cylinder length=0.02 radius=0.035
- link front_right_wheel: geometry visual cylinder length=0.02 radius=0.035
- link rear_left_wheel: geometry visual cylinder length=0.02 radius=0.035
- link rear_right_wheel: geometry visual cylinder length=0.02 radius=0.035
Joints:
- added joint rear_axis_joint: type fixed, parent base_link, child rear_wheel_axis, origin xyz=-0.12 0 0
- added joint steering_joint: type revolute, parent base_link, child steering_link, origin xyz=0.12 0 0, axis 0 0 1, limit lower=-0.785 upper=0.785 effort=10 velocity=1
- joint front_left_wheel_joint: axis (none) -> 0 0 1; origin xyz=0.12 0.07 -0.045 rpy=-1.5708 0 0 -> xyz=0 0.06 -0.035 rpy=${pi/2} 0 0; parent base_link -> steering_link; type fixed -> continuous
- joint front_right_wheel_joint: axis (none) -> 0 0 1; origin xyz=0.12 -0.07 -0.045 rpy=-1.5708 0 0 -> xyz=0 -0.06 -0.035 rpy=${pi/2} 0 0; parent base_link -> steering_link; type fixed -> continuous
- joint rear_left_wheel_joint: axis (none) -> 0 0 1; origin xyz=-0.12 0.07 -0.045 rpy=-1.5708 0 0 -> xyz=0 0.06 -0.035 rpy=${pi/2} 0 0; parent base_link -> rear_wheel_axis; type fixed -> continuous
- joint rear_right_wheel_joint: axis (none) -> 0 0 1; origin xyz=-0.12 -0.07 -0.045 rpy=-1.5708 0 0 -> xyz=0 -0.06 -0.035 rpy=${pi/2} 0 0; parent base_link -> rear_wheel_axis; type fixed -> continuous

Commit message: :card_file_box:[Mod] URDF 수정정

File: src/my_slam/urdf/robot.urdf (robot description, URDF)
Before this commit: robot my_robot, 9 links, 8 joints
Joints:
- joint front_left_wheel_joint: origin xyz=0 0.06 -0.035 rpy=${pi/2} 0 0 -> xyz=0 0.06 -0.035 rpy=1.5708 0 0
- joint front_right_wheel_joint: origin xyz=0 -0.06 -0.035 rpy=${pi/2} 0 0 -> xyz=0 -0.06 -0.035 rpy=1.5708 0 0
- joint rear_left_wheel_joint: origin xyz=0 0.06 -0.035 rpy=${pi/2} 0 0 -> xyz=0 0.06 -0.035 rpy=1.5708 0 0
- joint rear_right_wheel_joint: origin xyz=0 -0.06 -0.035 rpy=${pi/2} 0 0 -> xyz=0 -0.06 -0.035 rpy=1.5708 0 0
